File: pcb_main/spora.kicad_pcb (KiCad board)
At the start: 6 copper layers, 16.8 x 18.4 mm, 67 parts, among them J1 DF12D-3.0-10DP-0.5V-81, J2 DF12D-3.0-10DP-0.5V-81, SW1 SIDE_SW, U1 TPS2115a, U2 TPS82740B, U3 MCP73831, U4 MKL03Z32CAF4R, U5 LBCA2HNZYZ-711, U6 MPU-9250, Y1 32,768 kHz

Commit message: moved Vcc pin a few blocks
Parts:
- moved TP1 1.26 mm to (88.8, 70.1)
Routing:
- net /Power Supply/VBUS: track 13.2 -> 14.6 mm
